File: eagle/deadlocks2.brd (EAGLE design)
At the start: 78.4 x 120.2 mm, 18 parts, among them J1 6_PIN_SERIAL_CABLEPTH, U1 328P

Commit message: Finalized for prototype
Routing:
- net GND: track 0.00 -> 174.4 mm
- net N$20: track 0.00 -> 128.2 mm
- net VCC: track 0.00 -> 126.4 mm
- net N$21: track 0.00 -> 98.6 mm
- net N$18: track 0.00 -> 71.1 mm
- net N$1: track 0.00 -> 69.3 mm
- net N$10: track 0.00 -> 64.8 mm
- net N$14: track 0.00 -> 64.3 mm
- net N$15: track 0.00 -> 58.4 mm
- net N$24: track 0.00 -> 57.4 mm
- net N$8: track 0.00 -> 55.6 mm, vias 0 -> 1
- net N$9: track 0.00 -> 55.4 mm
- net N$7: track 0.00 -> 53.6 mm, vias 0 -> 1
- net N$22: track 0.00 -> 52.6 mm, vias 0 -> 1
- net N$25: track 0.00 -> 48.2 mm, vias 0 -> 1
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Other:
- board text added: "@DEAD10C5 DEFCON 26 #Badgelife"
- board text added: "@TheDevilsVoice @mzbat @p0lr_"
