File: eagle/deadlocks.sch (EAGLE design)
At the start: 18 parts, among them J1 6_PIN_SERIAL_CABLEPTH, U1 328P

Commit message: Re-arranged components, added a power input, and fixed the gerbers so Seeed can manufacture the prototypes.
Parts:
- added POWER: (no value), SparkFun-Connectors:CONN_02
- renumbered ISP1 to ISP
Connections:
- net GND: now also POWER.2
- net VCC: now also POWER.1
Changed lines of the file:
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@@
 <part name="GND5" library="supply1" library_urn="urn:adsk.eagle:library:371" deviceset="GND" device=""/>
 <part name="P+3" library="supply1" library_urn="urn:adsk.eagle:library:371" deviceset="VCC" device=""/>
-<part name="ISP1" library="adafruit" library_urn="urn:adsk.eagle:library:420" deviceset="AVRISP" device="-6"/>
+<part name="ISP" library="adafruit" library_urn="urn:adsk.eagle:library:420" deviceset="AVRISP" device="-6"/>
 <part name="P+4" library="supply1" library_urn="urn:adsk.eagle:library:371" deviceset="VCC" device=""/>
 <part name="GND7" library="supply1" library_urn="urn:adsk.eagle:library:371" deviceset="GND" device=""/>
 <part name="CLOCK" library="SparkFun-Clocks" library_urn="urn:adsk.eagle:library:511" deviceset="RESONATOR" device="PTH-7.6X3.8" package3d_urn="urn:adsk.eagle:package:37527/1" value="16MHz"/>
 <part name="RESISTOR" library="SparkFun-Connectors" library_urn="urn:adsk.eagle:library:513" deviceset="CONN_07" device="" package3d_urn="urn:adsk.eagle:package:38129/1" value="10Ohm"/>
+<part name="POWER" library="SparkFun-Connectors" library_urn="urn:adsk.eagle:library:513" deviceset="CONN_02" device="" package3d_urn="urn:adsk.eagle:package:38039/1"/>
+<part name="GND8" library="supply1" library_urn="urn:adsk.eagle:library:371" deviceset="GND" device=""/>
+<part name="P+6" library="supply1" library_urn="urn:adsk.eagle:library:371" deviceset="VCC" device=""/>
 </parts>
 <sheets>
@@
 <instance part="GND5" gate="1" x="152.4" y="25.4"/>
 <instance part="P+3" gate="VCC" x="-12.7" y="88.9"/>
-<instance part="ISP1" gate="G$1" x="15.24" y="-22.86"/>
+<instance part="ISP" gate="G$1" x="15.24" y="-22.86"/>
 <instance part="P+4" gate="VCC" x="35.56" y="-10.16"/>
 <instance part="GND7" gate="1" x="35.56" y="-33.02"/>
 <instance part="CLOCK" gate="G$1" x="17.78" y="48.26" rot="R270"/>
 <instance part="RESISTOR" gate="G$1" x="88.9" y="-40.64" rot="R90"/>
+<instance part="POWER" gate="G$1" x="137.16" y="10.16"/>
+<instance part="GND8" gate="1" x="157.48" y="5.08"/>
+<instance part="P+6" gate="VCC" x="147.32" y="5.08" rot="R180"/>
 </instances>
 <busses>
@@
 <segment>
 <pinref part="GND7" gate="1" pin="GND"/>
-<pinref part="ISP1" gate="G$1" pin="GND"/>
+<pinref part="ISP" gate="G$1" pin="GND"/>
 <wire x1="35.56" y1="-30.48" x2="35.56" y2="-25.4" width="0.1524" layer="91"/>
 <wire x1="35.56" y1="-25.4" x2="30.48" y2="-25.4" width="0.1524" layer="91"/>
@@
 <wire x1="93.98" y1="-35.56" x2="93.98" y2="-33.02" width="0.1524" layer="91"/>
 <wire x1="93.98" y1="-33.02" x2="111.76" y2="-33.02" width="0.1524" layer="91"/>
+</segment>
+<segment>
+<pinref part="POWER" gate="G$1" pin="2"/>
+<pinref part="GND8" gate="1" pin="GND"/>
+<wire x1="144.78" y1="12.7" x2="157.48" y2="12.7" width="0.1524" layer="91"/>
+<wire x1="157.48" y1="12.7" x2="157.48" y2="7.62" width="0.1524" layer="91"/>
 </segment>
 </net>
@@
 </segment>
 <segment>
-<pinref part="ISP1" gate="G$1" pin="VCC"/>
+<pinref part="ISP" gate="G$1" pin="VCC"/>
 <pinref part="P+4" gate="VCC" pin="VCC"/>
 <wire x1="30.48" y1="-20.32" x2="35.56" y2="-20.32" width="0.1524" layer="91"/>
 <wire x1="35.56" y1="-20.32" x2="35.56" y2="-12.7" width="0.1524" layer="91"/>
+</segment>
+<segment>
+<pinref part="POWER" gate="G$1" pin="1"/>
+<pinref part="P+6" gate="VCC" pin="VCC"/>
+<wire x1="144.78" y1="10.16" x2="147.32" y2="10.16" width="0.1524" layer="91"/>
+<wire x1="147.32" y1="10.16" x2="147.32" y2="7.62" width="0.1524" layer="91"/>
 </segment>
 </net>
@@
 <pinref part="U1" gate="G$1" pin="PC6(/RESET)"/>
 <wire x1="15.24" y1="76.2" x2="17.78" y2="76.2" width="0.1524" layer="91"/>
-<pinref part="ISP1" gate="G$1" pin="RST"/>
+<pinref part="ISP" gate="G$1" pin="RST"/>
 <wire x1="17.78" y1="76.2" x2="22.86" y2="76.2" width="0.1524" layer="91"/>
 <wire x1="2.54" y1="-25.4" x2="-12.7" y2="-25.4" width="0.1524" layer="91"/>
@@
 <net name="N$9" class="0">
 <segment>
-<pinref part="ISP1" gate="G$1" pin="MISO"/>
+<pinref part="ISP" gate="G$1" pin="MISO"/>
 <wire x1="2.54" y1="-20.32" x2="0" y2="-20.32" width="0.1524" layer="91"/>
 <wire x1="0" y1="-20.32" x2="0" y2="2.54" width="0.1524" layer="91"/>
@@
 <wire x1="101.6" y1="22.86" x2="101.6" y2="-17.78" width="0.1524" layer="91"/>
 <pinref part="D6" gate="G$1" pin="A"/>
-<pinref part="ISP1" gate="G$1" pin="MOSI"/>
+<pinref part="ISP" gate="G$1" pin="MOSI"/>
 <wire x1="30.48" y1="-22.86" x2="45.72" y2="-22.86" width="0.1524" layer="91"/>
 <wire x1="45.72" y1="-22.86" x2="45.72" y2="0" width="0.1524" layer="91"/>
@@
 <net name="N$24" class="0">
 <segment>
-<pinref part="ISP1" gate="G$1" pin="SCK"/>
+<pinref part="ISP" gate="G$1" pin="SCK"/>
 <wire x1="2.54" y1="-22.86" x2="-2.54" y2="-22.86" width="0.1524" layer="91"/>
 <wire x1="-2.54" y1="-22.86" x2="-2.54" y2="5.08" width="0.1524" layer="91"/>

Commit message: A few more mods with new gerbers
Parts:
- removed C3: 0.1uF, SparkFun-Capacitors:0.1UF-KIT-EZ-50V-20%
- added C1: 0.1uF, adafruit:C-US025-024X044
- RESISTOR: value 10Ohm -> 330 Ohm
Connections:
- net N$10: now also C1.1; no longer C3.1
- net N$11: now also C1.2; no longer C3.2
