File: eagle/deadlocks3.brd (EAGLE design)
At the start: 78.4 x 120.2 mm, 24 parts, among them U1 328P

Commit message: More updates to the board and the code
Parts:
- OLED: value (none) -> OLED
- renumbered I2C to OLED
Connections:
- net GND: now also OLED.4; no longer OLED.3
- net N$10: now also OLED.3; no longer OLED.4
Routing:
- net N$24: track 49.1 -> 156.1 mm, vias 2 -> 0
- net N$9: track 147.5 -> 54.4 mm
- net N$1: track 163.4 -> 89.6 mm, vias 4 -> 1
- net GND: track 239.4 -> 287.9 mm, vias 3 -> 1
- net N$28: track 160.7 -> 116.3 mm, vias 1 -> 5
- net N$20: track 96.6 -> 134.8 mm, vias 3 -> 1
- net N$5: track 65.8 -> 101.1 mm, vias 3 -> 4
- net N$8: track 89.5 -> 59.9 mm, vias 3 -> 2
- net N$18: track 102.1 -> 72.7 mm, vias 3 -> 0
- net N$7: track 61.0 -> 88.5 mm
- net N$15: track 78.8 -> 51.5 mm, vias 0 -> 1
- net N$17: track 33.8 -> 14.8 mm, vias 2 -> 0
- net N$10: track 117.3 -> 136.0 mm, vias 0 -> 1
- net N$26: track 136.2 -> 152.5 mm
- net N$11: track 105.0 -> 91.1 mm
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