File: eagle/deadlocks3.sch (EAGLE design)
At the start: 24 parts, among them U1 328P

Commit message: More updates to the board and the code
Parts:
- OLED: value (none) -> OLED
- renumbered I2C to OLED
Connections:
- net GND: now also OLED.4; no longer OLED.3
- net N$10: now also OLED.3; no longer OLED.4
Changed lines of the file:
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@@
 </variantdefs>
 <classes>
-<class number="0" name="default" width="0" drill="0">
+<class number="0" name="default" width="0.127" drill="0">
 <clearance class="0" value="0.254"/>
 </class>
@@
 <part name="P+6" library="supply1" library_urn="urn:adsk.eagle:library:371" deviceset="VCC" device=""/>
 <part name="C1" library="adafruit" library_urn="urn:adsk.eagle:library:420" deviceset="C-US" device="025-024X044" value="0.1uF"/>
-<part name="I2C" library="SparkFun-Connectors" library_urn="urn:adsk.eagle:library:513" deviceset="CONN_04" device="" package3d_urn="urn:adsk.eagle:package:38085/1"/>
+<part name="OLED" library="SparkFun-Connectors" library_urn="urn:adsk.eagle:library:513" deviceset="CONN_04" device="" package3d_urn="urn:adsk.eagle:package:38085/1" value="OLED"/>
 <part name="R2" library="SparkFun-Resistors" library_urn="urn:adsk.eagle:library:532" deviceset="10KOHM" device="-HORIZ-1/4W-1%" package3d_urn="urn:adsk.eagle:package:39658/1" value="3.6k"/>
 <part name="R3" library="SparkFun-Resistors" library_urn="urn:adsk.eagle:library:532" deviceset="10KOHM" device="-HORIZ-1/4W-1%" package3d_urn="urn:adsk.eagle:package:39658/1" value="10k"/>
@@
 <instance part="P+6" gate="VCC" x="134.62" y="17.78"/>
 <instance part="C1" gate="G$1" x="10.16" y="76.2" rot="R90"/>
-<instance part="I2C" gate="G$1" x="144.78" y="-40.64" rot="R90"/>
+<instance part="OLED" gate="G$1" x="144.78" y="-40.64" rot="R90"/>
 <instance part="R2" gate="G$1" x="119.38" y="-25.4" rot="R270"/>
 <instance part="R3" gate="G$1" x="127" y="-25.4" rot="R270"/>
@@
 <pinref part="GND2" gate="1" pin="GND"/>
 <wire x1="127" y1="-20.32" x2="127" y2="-17.78" width="0.1524" layer="91"/>
-<pinref part="I2C" gate="G$1" pin="3"/>
-<wire x1="142.24" y1="-35.56" x2="142.24" y2="-20.32" width="0.1524" layer="91"/>
-<wire x1="142.24" y1="-20.32" x2="127" y2="-20.32" width="0.1524" layer="91"/>
 <junction x="127" y="-20.32"/>
 <pinref part="BADGELIFE1" gate="G$1" pin="4"/>
 <wire x1="162.56" y1="-35.56" x2="162.56" y2="-20.32" width="0.1524" layer="91"/>
-<wire x1="162.56" y1="-20.32" x2="142.24" y2="-20.32" width="0.1524" layer="91"/>
-<junction x="142.24" y="-20.32"/>
+<wire x1="162.56" y1="-20.32" x2="139.7" y2="-20.32" width="0.1524" layer="91"/>
 <pinref part="BADGELIFE2" gate="G$1" pin="4"/>
+<wire x1="139.7" y1="-20.32" x2="127" y2="-20.32" width="0.1524" layer="91"/>
 <wire x1="182.88" y1="-35.56" x2="182.88" y2="-20.32" width="0.1524" layer="91"/>
 <wire x1="182.88" y1="-20.32" x2="162.56" y2="-20.32" width="0.1524" layer="91"/>
 <junction x="162.56" y="-20.32"/>
+<pinref part="OLED" gate="G$1" pin="4"/>
+<wire x1="139.7" y1="-35.56" x2="139.7" y2="-20.32" width="0.1524" layer="91"/>
+<junction x="139.7" y="-20.32"/>
 </segment>
 </net>
@@
 <wire x1="119.38" y1="-33.02" x2="119.38" y2="-30.48" width="0.1524" layer="91"/>
 <pinref part="BADGELIFE1" gate="G$1" pin="1"/>
-<wire x1="127" y1="-33.02" x2="139.7" y2="-33.02" width="0.1524" layer="91"/>
-<wire x1="139.7" y1="-33.02" x2="170.18" y2="-33.02" width="0.1524" layer="91"/>
+<wire x1="127" y1="-33.02" x2="142.24" y2="-33.02" width="0.1524" layer="91"/>
+<wire x1="142.24" y1="-33.02" x2="170.18" y2="-33.02" width="0.1524" layer="91"/>
 <wire x1="170.18" y1="-33.02" x2="170.18" y2="-35.56" width="0.1524" layer="91"/>
 <junction x="127" y="-33.02"/>
@@
 <wire x1="190.5" y1="-33.02" x2="190.5" y2="-35.56" width="0.1524" layer="91"/>
 <junction x="170.18" y="-33.02"/>
-<pinref part="I2C" gate="G$1" pin="4"/>
-<wire x1="139.7" y1="-35.56" x2="139.7" y2="-33.02" width="0.1524" layer="91"/>
-<junction x="139.7" y="-33.02"/>
+<pinref part="OLED" gate="G$1" pin="3"/>
+<wire x1="142.24" y1="-35.56" x2="142.24" y2="-33.02" width="0.1524" layer="91"/>
+<junction x="142.24" y="-33.02"/>
 </segment>
 </net>
 <net name="N$26" class="0">
 <segment>
-<pinref part="I2C" gate="G$1" pin="1"/>
+<pinref part="OLED" gate="G$1" pin="1"/>
 <wire x1="147.32" y1="-35.56" x2="147.32" y2="-2.54" width="0.1524" layer="91"/>
 <wire x1="147.32" y1="-2.54" x2="121.92" y2="-2.54" width="0.1524" layer="91"/>
@@
 <net name="N$28" class="0">
 <segment>
-<pinref part="I2C" gate="G$1" pin="2"/>
+<pinref part="OLED" gate="G$1" pin="2"/>
 <wire x1="144.78" y1="-35.56" x2="144.78" y2="-5.08" width="0.1524" layer="91"/>
 <wire x1="144.78" y1="-5.08" x2="119.38" y2="-5.08" width="0.1524" layer="91"/>
@@
 </sheet>
 </sheets>
-<errors>
-</errors>
 </schematic>
 </drawing>
